File: Hardware/matrixSAO/LED_Matrix.kicad_sch (KiCad schematic)
At the start: 161 parts

Commit message: update
Parts:
- removed D10, D106, D107, D108, D109, D11, D110, D111, D112, D12, D120, D121, D122, D123, D124, D125, D126, D13, D134, D135, D136, D137, D138, D139, D14, D140, D148, D149, D150, D151, D152, D153, D154, D155, D156, D157, D158, D159, D160, D161, D22, D23, D24, D25, D26, D27, D28, D36, D37, D38, D39, D40, D41, D42, D50, D51, D52, D53, D54, D55, D56, D64, D65, D66, D67, D68, D69, D70, D78, D79, D8, D80, D81, D82, D83, D84, D9, D92, D93, D94, D95, D96, D97, D98: LED, symbol Device:LED

Commit message: Order at JLCPPCB
Parts:
- D1, D100, D101, D102, D103, D104, D105, D113, D114, D115, D116, D117, D118, D119, D127, D128, D129, D130, D131, D132, D133, D141, D142, D143, D144, D145, D146, D147, D15, D16, D17, D18, D19, D2, D20, D21, D29, D3, D30, D31, D32, D33, D34, D35, D4, D43, D44, D45, D46, D47, D48, D49, D5, D57, D58, D59, D6, D60, D61, D62, D63, D7, D71, D72, D73, D74, D75, D76, D77, D85, D86, D87, D88, D89, D90, D91, D99: LCSC (none) -> C965793
