File: Hardware/matrixSAO/MCU.kicad_sch (KiCad schematic)
At the start: 0 parts

Commit message: some work
Parts:
- added C1: C, dipolMods:C_0402_min, symbol Device:C
- added U1: CH32V003FxUx, Package_DFN_QFN:QFN-20-1EP_3x3mm_P0.4mm_EP1.65x1.65mm, symbol MCU_WCH_CH32V0:CH32V003FxUx
Connections:
- new net +3.3V: C1.2, U1.6 (VDD)
- new net A1: U1.2 (PA1)
- new net A2: U1.3 (PA2)
- new net C0: U1.7 (PC0)
- new net C3: U1.10 (PC3)
- new net C4: U1.11 (PC4)
- new net C5: U1.12 (PC5)
- new net C6: U1.13 (PC6)
- new net C7: U1.14 (PC7)
- new net D0: U1.5 (PD0)
- new net D2: U1.16 (PD2)
- new net D3: U1.17 (PD3)
- new net D4: U1.18 (PD4)
- new net D5: U1.19 (PD5)
- new net D6: U1.20 (PD6)
- new net D7: U1.1 (PD7)
- new net GND: C1.1, U1.21 (VSS), U1.4 (VSS)
- new net SCL: U1.9 (PC2)
- new net SDA: U1.8 (PC1)
- new net SWDIO: U1.15 (PD1)

Commit message: Order at JLCPPCB
Parts:
- C1: LCSC (none) -> C16772
- U1: LCSC (none) -> C5299908
Changed lines of the file:
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@@
+			)
+		)
+		(property "LCSC" "C16772"
+			(at 146.05 50.8 0)
+			(effects
+				(font
+					(size 1.27 1.27)
+				)
+				(hide yes)
 			)
 		)
@@
 			(at 152.4 71.12 0)
 			(effects
+				(font
+					(size 1.27 1.27)
+				)
+				(hide yes)
+			)
+		)
+		(property "LCSC" "C5299908"
+			(at 152.4 71.12 0)
+			(effects
