File: Hardware/matrixSAO/matrixSAO.kicad_pcb (KiCad board)
At the start: 2 copper layers, 17 x 18.5 mm, 81 parts, among them J1 Conn_02x03_Odd_Even, U1 CH32V003FxUx

Commit message: update
Parts:
- added REF**: deko0402silk, ownMisc:deko0402silk, F.Cu at (70.5, 131.5)
- added REF**: deko0402silk, ownMisc:deko0402silk, F.Cu at (70.5, 130.0)
- added REF**: deko0402silk, ownMisc:deko0402silk, F.Cu at (70.5, 128.5)
- added REF**: deko0402silk, ownMisc:deko0402silk, F.Cu at (73.5, 128.5)
- added REF**: deko0402silk, ownMisc:deko0402silk, F.Cu at (73.5, 130.0)
- added REF**: deko0402silk, ownMisc:deko0402silk, F.Cu at (70.5, 127.0)
- added REF**: deko0402silk, ownMisc:deko0402silk, F.Cu at (72.0, 131.5)
- added REF**: deko0402silk, ownMisc:deko0402silk, F.Cu at (72.0, 130.0)
- added REF**: deko0402silk, ownMisc:deko0402silk, F.Cu at (73.5, 127.0)
- added REF**: deko0402silk, ownMisc:deko0402silk, F.Cu at (73.5, 131.5)
Connections:
- U1 pad 2: /MCU/A1 -> /IO1
Routing:
- net GND: track 22.0 -> 2.18 mm, vias 1 -> 19
- net /LED-Matrix/8: track 32.0 -> 48.2 mm, vias 5 -> 10
- net +3.3V: track 13.0 -> 24.5 mm, vias 1 -> 3
- net /LED-Matrix/6: track 29.5 -> 39.6 mm, vias 4 -> 8
- net /LED-Matrix/E: track 9.63 -> 19.2 mm, vias 1 -> 5
- net /LED-Matrix/F: track 5.29 -> 9.96 mm, vias 0 -> 3
- net /LED-Matrix/4: track 27.3 -> 31.9 mm
- net /IO1: track 0.00 -> 1.76 mm
- net /IO0: track 7.76 -> 9.33 mm
- net /LED-Matrix/7: track 24.1 -> 25.5 mm
- net /SCL: track 8.91 -> 7.73 mm
- added copper zone on B.Cu, net GND
- added copper zone on F.Cu, net GND

Commit message: Order at JLCPPCB
Parts:
- REF** (x6): value deko0402silk -> deko0402Mask; footprint ownMisc:deko0402silk -> ownMisc:deko0402Mask
