File: Hardware/matrixSAO/matrixSAO.kicad_sch (KiCad schematic)
At the start: 1 part, among them J1 Conn_02x03_Odd_Even

Commit message: some work
Parts:
- J1: footprint (none) -> Connector_IDC:IDC-Header_2x03_P2.54mm_Vertical
Connections:
- net VCC: now reaches J1.1 (Pin_1)
- net GND: now reaches J1.2 (Pin_2)
- net SDA: now reaches J1.3 (Pin_3)
- net SCL: now reaches J1.4 (Pin_4)
- net IO1: now reaches J1.5 (Pin_5)
- net IO0: now reaches J1.6 (Pin_6)
Other:
- sheet MCU ports: added A1, A2, C0, C3, C4, C5, C6, C7, D0, D2, D3, D4, D5, D6, D7, SCL, SDA, SWDIO; removed none
- moved on the sheet: J1

Commit message: update
Parts:
- added C2: C, dipolMods:C_0402_min, symbol Device:C
- added J2: Conn_01x03, Connector_PinHeader_1.27mm:PinHeader_1x03_P1.27mm_Vertical, symbol Connector_Generic:Conn_01x03
Connections:
- net GND: now also C2.1
- net VCC renamed +3.3V
- net +3.3V: now also C2.2
Other:
- sheet LED-Matrix ports: added none; removed 9, B

Commit message: update
Parts:
- removed J2: Conn_01x03, Connector_PinHeader_1.27mm:PinHeader_1x03_P1.27mm_Vertical, symbol Connector_Generic:Conn_01x03
Other:
- moved on the sheet: C2
Changed lines of the file:
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@@
+	(wire
+		(pts
+			(xy 88.9 92.71) (xy 88.9 96.52)
+		)
+		(stroke
+			(width 0)
+			(type default)
+		)
+	)
 	(wire
 		(pts
@@
 		(pts
 			(xy 123.19 87.63) (xy 123.19 80.01)
+		)
+		(stroke
+			(width 0)
+			(type default)
+		)
+	)
+	(wire
+		(pts
+			(xy 88.9 96.52) (xy 129.54 96.52)
 		)
 		(stroke
@@
 	(symbol
 		(lib_id "power:+3.3V")
-		(at 118.11 97.79 0)
+		(at 99.06 119.38 0)
 		(unit 1)
 		(exclude_from_sim no)
@@
 		(fields_autoplaced yes)
 		(property "Reference" "#PWR07"
-			(at 118.11 101.6 0)
+			(at 99.06 123.19 0)
 			(effects
 				(font
@@
 		)
 		(property "Value" "+3.3V"
-			(at 118.11 92.71 0)
+			(at 99.06 114.3 0)
 			(effects
 				(font
@@
 		)
 		(property "Footprint" ""
-			(at 118.11 97.79 0)
+			(at 99.06 119.38 0)
 			(effects
 				(font
@@
 		)
 		(property "Datasheet" ""
-			(at 118.11 97.79 0)
+			(at 99.06 119.38 0)
 			(effects
 				(font
@@
 		)
 		(property "Description" "Power symbol creates a global label with name \"+3.3V\""
-			(at 118.11 97.79 0)
+			(at 99.06 119.38 0)
 			(effects
 				(font
@@
 	(symbol
 		(lib_id "power:GND")
-		(at 118.11 105.41 0)
+		(at 99.06 127 0)
 		(unit 1)
 		(exclude_from_sim no)
@@
 		(fields_autoplaced yes)
 		(property "Reference" "#PWR06"
-			(at 118.11 111.76 0)
+			(at 99.06 133.35 0)
 			(effects
 				(font
@@
 		)
 		(property "Value" "GND"
-			(at 118.11 110.49 0)
+			(at 99.06 132.08 0)
 			(effects
 				(font
@@
 		)
 		(property "Footprint" ""
-			(at 118.11 105.41 0)
+			(at 99.06 127 0)
 			(effects
 				(font
@@
 		)
 		(property "Datasheet" ""
-			(at 118.11 105.41 0)
+			(at 99.06 127 0)
 			(effects
 				(font
@@
 		)
 		(property "Description" "Power symbol creates a global label with name \"GND\" , ground"
-			(at 118.11 105.41 0)
+			(at 99.06 127 0)
 			(effects
 				(font
@@
 				(path "/97d6d41c-c50e-47f0-85e1-8023869e228c"
 					(reference "#PWR06")
-					(unit 1)
-				)
-			)
-		)
-	)
-	(symbol
-		(lib_id "Connector_Generic:Conn_01x03")
-		(at 100.33 107.95 270)
-		(unit 1)
-		(exclude_from_sim no)
-		(in_bom yes)
-		(on_board yes)
-		(dnp no)
-		(fields_autoplaced yes)
-		(property "Reference" "J2"
-			(at 105.41 106.6799 90)
-			(effects
-				(font
-					(size 1.27 1.27)
-				)
-				(justify left)
-			)
-		)
-		(property "Value" "Conn_01x03"
-			(at 105.41 109.2199 90)
-			(effects
-				(font
-					(size 1.27 1.27)
-				)
-				(justify left)
-			)
-		)
-		(property "Footprint" "Connector_PinHeader_1.27mm:PinHeader_1x03_P1.27mm_Vertical"
-			(at 100.33 107.95 0)
-			(effects
-				(font
-					(size 1.27 1.27)
-				)
-				(hide yes)
-			)
-		)
-		(property "Datasheet" "~"
-			(at 100.33 107.95 0)
-			(effects
-				(font
-					(size 1.27 1.27)
-				)
-				(hide yes)
-			)
-		)
-		(property "Description" "Generic connector, single row, 01x03, script generated (kicad-library-utils/schlib/autogen/connector/)"
-			(at 100.33 107.95 0)
-			(effects
-				(font
-					(size 1.27 1.27)
-				)
-				(hide yes)
-			)
-		)
-		(pin "2"
-		)
-		(pin "1"
-		)
-		(pin "3"
-		)
-		(instances
-			(project ""
-				(path "/97d6d41c-c50e-47f0-85e1-8023869e228c"
-					(reference "J2")
 					(unit 1)
 				)
@@
 	(symbol
 		(lib_id "Device:C")
-		(at 118.11 101.6 180)
+		(at 99.06 123.19 180)
 		(unit 1)
 		(exclude_from_sim no)
@@
 		(fields_autoplaced yes)
 		(property "Reference" "C2"
-			(at 121.92 100.3299 0)
+			(at 102.87 121.9199 0)
 			(effects
 				(font
@@
 		)
 		(property "Value" "C"
-			(at 121.92 102.8699 0)
+			(at 102.87 124.4599 0)
 			(effects
 				(font
@@
 		)
 		(property "Footprint" "dipolMods:C_0402_min"
-			(at 117.1448 97.79 0)
+			(at 98.0948 119.38 0)
 			(effects
 				(font
@@
 		)
 		(property "Datasheet" "~"
-			(at 118.11 101.6 0)
+			(at 99.06 123.19 0)
 			(effects
 				(font
@@
 		)
 		(property "Description" "Unpolarized capacitor"
-			(at 118.11 101.6 0)
+			(at 99.06 123.19 0)
 			(effects
 				(font
@@
 		)
 		(pin "A1" input
-			(at 129.54 99.06 180)
+			(at 129.54 96.52 180)
 			(effects
 				(font
@@
 		)
 		(pin "A2" input
-			(at 137.16 85.09 90)
-			(effects
-				(font
-					(size 1.27 1.27)
-				)
-				(justify right)
-			)
-		)
+			(at 129.54 101.6 180)
+			(effects
+				(font
+					(size 1.27 1.27)
+				)
+				(justify left)
+			)
+		)

Commit message: Order at JLCPPCB
Parts:
- C2: LCSC (none) -> C16772
- J1: LCSC (none) -> C4749192
Changed lines of the file:
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@@
+			)
+		)
+		(property "LCSC" "C4749192"
+			(at 99.06 90.17 0)
+			(effects
+				(font
+					(size 1.27 1.27)
+				)
+				(hide yes)
 			)
 		)
@@
 			(at 99.06 123.19 0)
 			(effects
+				(font
+					(size 1.27 1.27)
+				)
+				(hide yes)
+			)
+		)
+		(property "LCSC" "C16772"
+			(at 99.06 123.19 0)
+			(effects
